Commit message: Launch file setup

File: src/my_robot_controller/description/my_robot.urdf (robot description, URDF)
Before this commit: robot slam_robot, 3 links, 1 joints
Links:
- removed link left_wheel
- added link left_wheel_back; visual cylinder length=0.014 radius=0.045
- added link left_wheel_front; visual cylinder length=0.014 radius=0.045
- added link right_wheel_back; visual cylinder length=0.014 radius=0.045
- added link right_wheel_front; visual cylinder length=0.014 radius=0.045
Joints:
- added joint base_left_wheel_back_joint: type fixed, parent base_link, child left_wheel_back, origin xyz=-0.0625 0.082 0.02 rpy=0 0 0, axis 0 1 0
- added joint base_left_wheel_front_joint: type fixed, parent base_link, child left_wheel_front, origin xyz=0.0625 0.082 0.02 rpy=0 0 0, axis 0 1 0
- added joint base_right_wheel_back_joint: type fixed, parent base_link, child right_wheel_back, origin xyz=-0.0625 -0.082 0.02 rpy=0 0 0, axis 0 1 0
- added joint base_right_wheel_front_joint: type fixed, parent base_link, child right_wheel_front, origin xyz=0.0625 -0.082 0.02 rpy=0 0 0, axis 0 1 0
- joint base_lidar_joint: origin xyz=0.07 0 0.1125 rpy=0 0 0 -> xyz=-0.07 0 0.1125 rpy=0 0 0

Commit message: 27.05.24 Changes

File: src/my_robot_controller/description/my_robot.urdf (robot description, URDF)
Before this commit: robot slam_robot, 6 links, 5 joints
Links:
- added link base_footprint
Joints:
- added joint base_joint: type fixed, parent base_footprint, child base_link, origin xyz=0 0 0.025 rpy=0 0 0
- joint base_left_wheel_back_joint: origin xyz=-0.0625 0.082 0.02 rpy=0 0 0 -> xyz=0.0625 -0.082 0.02 rpy=0 0 0
- joint base_left_wheel_front_joint: origin xyz=0.0625 0.082 0.02 rpy=0 0 0 -> xyz=-0.0625 -0.082 0.02 rpy=0 0 0
- joint base_lidar_joint: origin xyz=-0.07 0 0.1125 rpy=0 0 0 -> xyz=0.07 0 0.1125 rpy=0 0 0
- joint base_right_wheel_back_joint: origin xyz=-0.0625 -0.082 0.02 rpy=0 0 0 -> xyz=0.0625 0.082 0.02 rpy=0 0 0
- joint base_right_wheel_front_joint: origin xyz=0.0625 -0.082 0.02 rpy=0 0 0 -> xyz=-0.0625 0.082 0.02 rpy=0 0 0
